Commit message: feat(bringup): 真机后端参数化并改用 async 500 Hz
- z1_ros2_control.xacro 拆出真机与 Gazebo 两块，关节列表提成共用宏以免漂移：
  只有真机块带 rw_rate="500" is_async="true" 与 <properties><async
  scheduling_policy="detached"/>，Gazebo 块保持原样（该后端有自己的组件，不能被
  绑到我们的 500 Hz 工作线程上）。已核对两条路径的渲染结果，Gazebo 侧不出现
  async/rw_rate/param。
- 把 z1_ctrl 链路参数暴露成 <hardware><param>：ctrl_ip、ctrl_port、own_port、
  activate_fsm_sequence、disconnect_timeout_ms、temperature_limit；xacro 参数与
  control.launch.py 的 launch 参数同名同默认值，两者需同步维护。
- 注释写明 500 是传输率而非控制率：controller_manager 的 update_rate 仍为 250，
  与 z1_ctrl 的伺服循环一致。

File: src/z1_description/urdf/z1.urdf.xacro (robot description, xacro)
@@ -13,4 +13,15 @@
     controllers_file  (string)      : controller_manager parameter file used by the
                                       gz_ros2_control plugin (Gazebo backend only)
+  xacro args for the real-arm backend (`hardware_plugin` != GazeboSimSystem);
+  they become <param> entries of the <hardware> block:
+    ctrl_ip                  (string) : z1_ctrl's host, loopback by default
+    ctrl_port                (int)    : the port z1_ctrl binds (8071)
+    own_port                 (int)    : the port we bind (8072)
+    activate_fsm_sequence    (string) : comma-separated FSM states to request on
+                                        activation ("JOINTCTRL")
+    disconnect_timeout_ms    (int)    : silence from z1_ctrl that counts as a
+                                        hardware error (200)
+    temperature_limit        (int)    : motor over-temperature limit in Celsius,
+                                        matching z1_controller's own 80 (80)
 -->
 <robot name="z1" xmlns:xacro="http://www.ros.org/wiki/xacro">
@@ -21,4 +32,10 @@
     <xacro:arg name="controllers_file"
                default="$(find z1_bringup)/config/z1_controllers.yaml"/>
+    <xacro:arg name="ctrl_ip" default="127.0.0.1"/>
+    <xacro:arg name="ctrl_port" default="8071"/>
+    <xacro:arg name="own_port" default="8072"/>
+    <xacro:arg name="activate_fsm_sequence" default="JOINTCTRL"/>
+    <xacro:arg name="disconnect_timeout_ms" default="200"/>
+    <xacro:arg name="temperature_limit" default="80"/>
     <xacro:include filename="$(find z1_description)/urdf/const.xacro"/>
     <xacro:include filename="$(find z1_description)/urdf/z1_body.xacro"/>
@@ -37,5 +54,11 @@
     <xacro:z1_body use_gripper="$(arg use_gripper)"/>
     <xacro:z1_ros2_control use_gripper="$(arg use_gripper)"
-                           hardware_plugin="$(arg hardware_plugin)"/>
+                           hardware_plugin="$(arg hardware_plugin)"
+                           ctrl_ip="$(arg ctrl_ip)"
+                           ctrl_port="$(arg ctrl_port)"
+                           own_port="$(arg own_port)"
+                           activate_fsm_sequence="$(arg activate_fsm_sequence)"
+                           disconnect_timeout_ms="$(arg disconnect_timeout_ms)"
+                           temperature_limit="$(arg temperature_limit)"/>
     <xacro:z1_gz_ros2_control hardware_plugin="$(arg hardware_plugin)"
                               controllers_file="$(arg controllers_file)"/>

File: src/z1_description/urdf/z1_ros2_control.xacro (robot description, xacro)
@@ -14,4 +14,7 @@
   The gripper keeps its position interface: it is driven by a position
   controller (GripperActionController) on every backend.
+  Only the real-arm block is async. `gz_ros2_control` builds its own component
+  and must not be forced onto our 500 Hz worker thread; keeping the two blocks
+  apart also keeps the Gazebo path's URDF free of parameters it would ignore.
 -->
 <robot xmlns:xacro="http://www.ros.org/wiki/xacro">
@@ -25,28 +28,70 @@
         </joint>
     </xacro:macro>
-    <xacro:macro name="z1_ros2_control" params="use_gripper hardware_plugin">
-        <xacro:property name="arm_command_interface"
-                        value="${'effort' if hardware_plugin == 'gz_ros2_control/GazeboSimSystem' else 'position'}"/>
-        <ros2_control name="z1" type="system">
-            <hardware>
-                <plugin>${hardware_plugin}</plugin>
-            </hardware>
-            <xacro:z1_joint_interfaces joint_name="joint1"
-                                       command_interface="${arm_command_interface}"/>
-            <xacro:z1_joint_interfaces joint_name="joint2"
-                                       command_interface="${arm_command_interface}"/>
-            <xacro:z1_joint_interfaces joint_name="joint3"
-                                       command_interface="${arm_command_interface}"/>
-            <xacro:z1_joint_interfaces joint_name="joint4"
-                                       command_interface="${arm_command_interface}"/>
-            <xacro:z1_joint_interfaces joint_name="joint5"
-                                       command_interface="${arm_command_interface}"/>
-            <xacro:z1_joint_interfaces joint_name="joint6"
-                                       command_interface="${arm_command_interface}"/>
-            <xacro:if value="${use_gripper}">
-                <xacro:z1_joint_interfaces joint_name="jointGripper"
-                                           command_interface="position"/>
-            </xacro:if>
-        </ros2_control>
+    <!-- The joint set, shared by the two <ros2_control> blocks below so they
+         cannot drift apart. -->
+    <xacro:macro name="z1_ros2_control_joints" params="use_gripper command_interface">
+        <xacro:z1_joint_interfaces joint_name="joint1"
+                                   command_interface="${command_interface}"/>
+        <xacro:z1_joint_interfaces joint_name="joint2"
+                                   command_interface="${command_interface}"/>
+        <xacro:z1_joint_interfaces joint_name="joint3"
+                                   command_interface="${command_interface}"/>
+        <xacro:z1_joint_interfaces joint_name="joint4"
+                                   command_interface="${command_interface}"/>
+        <xacro:z1_joint_interfaces joint_name="joint5"
+                                   command_interface="${command_interface}"/>
+        <xacro:z1_joint_interfaces joint_name="joint6"
+                                   command_interface="${command_interface}"/>
+        <xacro:if value="${use_gripper}">
+            <xacro:z1_joint_interfaces joint_name="jointGripper"
+                                       command_interface="position"/>
+        </xacro:if>
+    </xacro:macro>
+    <xacro:macro name="z1_ros2_control"
+                 params="use_gripper hardware_plugin
+                         ctrl_ip ctrl_port own_port activate_fsm_sequence
+                         disconnect_timeout_ms:='200' temperature_limit:='80'">
+        <xacro:property name="is_gazebo"
+                        value="${hardware_plugin == 'gz_ros2_control/GazeboSimSystem'}"/>
+        <xacro:unless value="${is_gazebo}">
+            <!--
+              Real arm, via the official z1_ctrl process on the same machine.
+              rw_rate="500" is the transport rate, not the control rate: z1_ctrl's
+              ARMSDK loop runs at dt = 0.002 s and treats a cycle without an
+              incoming SendCmd as a timeout, so the client has to keep up at
+              500 Hz. controller_manager's own update_rate stays 250 to match the
+              arm's servo loop.
+              is_async + scheduling_policy="detached" makes ros2_control run this
+              component's read()/write() on its own worker thread at rw_rate,
+              which is where the UDP send/recv happens. That keeps the socket
+              syscalls off the controller_manager thread and avoids the official
+              ROS 1 driver's mistake of making the whole process SCHED_FIFO.
+            -->
+            <ros2_control name="z1" type="system" rw_rate="500" is_async="true">
+                <hardware>
+                    <plugin>${hardware_plugin}</plugin>
+                    <param name="ctrl_ip">${ctrl_ip}</param>
+                    <param name="ctrl_port">${ctrl_port}</param>
+                    <param name="own_port">${own_port}</param>
+                    <param name="activate_fsm_sequence">${activate_fsm_sequence}</param>
+                    <param name="disconnect_timeout_ms">${disconnect_timeout_ms}</param>
+                    <param name="temperature_limit">${temperature_limit}</param>
+                </hardware>
+                <properties>
+                    <async scheduling_policy="detached"/>
+                </properties>
+                <xacro:z1_ros2_control_joints use_gripper="${use_gripper}"
+                                             command_interface="position"/>
+            </ros2_control>
+        </xacro:unless>
+        <xacro:if value="${is_gazebo}">
+            <ros2_control name="z1" type="system">
+                <hardware>
+                    <plugin>${hardware_plugin}</plugin>
+                </hardware>
+                <xacro:z1_ros2_control_joints use_gripper="${use_gripper}"
+                                             command_interface="effort"/>
+            </ros2_control>
+        </xacro:if>
     </xacro:macro>
 </robot>
